Commit message: Rename rickshaw to tricycle

File: simulation/tricycle/model.urdf (robot description, URDF)
Before this commit: robot rickshaw, 5 links, 4 joints
Links:
- link base_link: geometry collision mesh filename=package://simulation/tricycle/meshes/collisions/bike.stl scale=0.001 0.001 0.001; visual mesh filename=package://simulation/tricycle/meshes/visuals/bike.stl scale=0.001 0.001 0.001
- link front_part: geometry collision mesh filename=package://simulation/tricycle/meshes/collisions/front_part.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 scale=0.001 0.001 0.001; visual mesh filename=package://simulation/tricycle/meshes/visuals/front_part.stl scale=0.001 0.001 0.001
- link left_wheel: geometry collision mesh filename=package://simulation/tricycle/meshes/visuals/left_wheel.stl scale=0.001 0.001 0.001; visual mesh filename=package://simulation/tricycle/meshes/visuals/left_wheel.stl scale=0.001 0.001 0.001
- link right_wheel: geometry collision mesh filename=package://simulation/tricycle/meshes/visuals/right_wheel.stl scale=0.001 0.001 0.001; visual mesh filename=package://simulation/tricycle/meshes/visuals/right_wheel.stl scale=0.001 0.001 0.001
- link wheel_back: geometry collision mesh filename=package://simulation/tricycle/meshes/visuals/wheel_back.stl scale=0.001 0.001 0.001; visual mesh filename=package://simulation/tricycle/meshes/visuals/wheel_back.stl scale=0.001 0.001 0.001
